Commit message: Add files via upload

File: robot/urdf/robot.urdf (robot description, URDF)
Before this commit: robot robot, 3 links, 2 joints
Links:
- link Body: mass 0.1421 -> 5.0
- link left_wheel: mass 0.013464 -> 2.0
- link right_wheel: mass 0.013464 -> 2.0
Joints:
- joint left_joint: type revolute -> continuous
- joint right_joint: type revolute -> continuous
